File: Larry_Load v3.kicad_pcb (KiCad board)
At the start: 2 copper layers, 207.8 x 101.6 mm, 91 parts, among them U1 TKISL21080DIH312Z-TK, U2 Opamp_Dual, U3 TPL5110, U4 TPS61222DCK

Commit message: Add files via upload
Fixed incorrect values for R31, R32
Parts:
- C5: value 100uF -> 47uF
- R31: value 10k -> 8.06k
- R32: value 10k -> 50k
- U1: value TKISL21080DIH312Z-TK -> REF3312AIDBZR
Changed lines of the file:
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@@
 			)
 		)
-		(property "Value" "10k"
+		(property "Value" "50k"
 			(at 0 -1.82 0)
 			(layer "B.Fab")
@@
 			)
 		)
-		(property "Value" "10k"
+		(property "Value" "8.06k"
 			(at -5.3 -0.25 0)
 			(layer "B.Fab")
@@
 			)
 		)
-		(property "Value" "TKISL21080DIH312Z-TK"
+		(property "Value" "REF3312AIDBZR"
 			(at 0 -2.4 0)
 			(layer "B.Fab")
@@
 			)
 		)
-		(property "Datasheet" "https://www.digikey.com/en/products/detail/renesas-electronics-corporation/ISL21080DIH312Z-TK/2551515"
+		(property "Datasheet" "https://www.digikey.com/en/products/detail/texas-instruments/REF3312AIDBZR/1900120"
 			(at 0 0 0)
 			(unlocked yes)
@@
 		(tags "capacitor handsolder")
 		(property "Reference" "C3"
-			(at 0 1.85 360)
+			(at 0 1.85 0)
 			(layer "B.SilkS")
 			(effects
@@
 		)
 		(property "Value" "10uF"
-			(at 0 -1.85 360)
+			(at 0 -1.85 0)
 			(layer "B.Fab")
 			(effects
@@
 		)
 		(fp_text user "${REFERENCE}"
-			(at 0 0 360)
+			(at 0 0 0)
 			(layer "B.Fab")
 			(effects
@@
 			)
 		)
-		(property "Value" "100uF"
+		(property "Value" "47uF"
 			(at 0 -4.349999 0)
 			(layer "B.Fab")
